Commit message: ur_description/urdf/ur3_chip_joint_limited_robot.urdf

File: ur_description/urdf/ur3_chip.urdf.xacro (robot description, xacro)
@@ -295,5 +295,5 @@
       <inertial>
         <origin xyz="0 0 0.004" rpy="0 0 0"/>
-        <mass value="0.1"/>
+        <mass value="1.2"/>
         <inertia ixx="0.0001"  ixy="0"  ixz="0" iyy="0.001" iyz="0" izz="0.001" />
      </inertial>
@@ -368,4 +368,5 @@
     <child link="${prefix}depth_camera"/>
   </joint>
+   <!--TODO add weight property for sensors -->
   </xacro:macro>
 </robot>
